Commit message: modify robot base tf

File: recon_bot_description/robot/robot.core.xacro (robot description, xacro)
@@ -16,45 +16,5 @@
     <origin xyz="0.0 0.0 0.0" rpy="0.0 0.0 3.14" />
   </link>
-  <link
-    name="Mobile_Base">
-    <inertial>
-      <origin
-        xyz="-0.000901764538349642 0.00289486712536702 -0.140394651236372"
-        rpy="0 0 0" />
-      <mass
-        value="12.2070426110808" />
-      <inertia
-        ixx="0.100263210317857"
-        ixy="0.000416138117875011"
-        ixz="1.90955749720013E-07"
-        iyy="0.0777870248737817"
-        iyz="-4.99662188803516E-08"
-        izz="0.15510236958373" />
-    </inertial>
-    <visual>
-      <origin
-        xyz="0 0 0"
-        rpy="0 0 0" />
-      <geometry>
-        <mesh
-          filename="package://recon_bot_description/meshes/Mobile_Base.STL" />
-      </geometry>
-      <material
-        name="">
-        <color
-          rgba="0.792156862745098 0.819607843137255 0.933333333333333 1" />
-      </material>
-    </visual>
-    <collision>
-      <origin
-        xyz="0 0 0"
-        rpy="0 0 0" />
-      <geometry>
-        <mesh
-          filename="package://recon_bot_description/meshes/Mobile_Base.STL" />
-      </geometry>
-    </collision>
-  </link>
-  <joint name="basefootprint_to_base" type="fixed">
+    <joint name="base_footprint_to_Mobile_Base" type="fixed">
     <parent link="base_footprint"/>
     <child link="Mobile_Base"/>
@@ -62,18 +22,58 @@
   </joint>
   <link
+    name="Mobile_Base">
+    <inertial>
+      <origin
+        xyz="0.00270794889201253 0.000926242394781646 -0.128115066829716"
+        rpy="0 0 0" />
+      <mass
+        value="13.0496430135498" />
+      <inertia
+        ixx="0.078428885336732"
+        ixy="-0.000424260125405416"
+        ixz="-4.99662127671641E-08"
+        iyy="0.101100659734584"
+        iyz="-1.90955777107521E-07"
+        izz="0.156190952643998" />
+    </inertial>
+    <visual>
+      <origin
+        xyz="0 0 0"
+        rpy="0 0 0" />
+      <geometry>
+        <mesh
+          filename="package://recon_bot_description/meshes/Mobile_Base.STL" />
+      </geometry>
+      <material
+        name="">
+        <color
+          rgba="0.792156862745098 0.819607843137255 0.933333333333333 1" />
+      </material>
+    </visual>
+    <collision>
+      <origin
+        xyz="0 0 0"
+        rpy="0 0 0" />
+      <geometry>
+        <mesh
+          filename="package://recon_bot_description/meshes/Mobile_Base.STL" />
+      </geometry>
+    </collision>
+  </link>
+  <link
     name="Wheel_LF">
     <inertial>
       <origin
-        xyz="-3.68604325448052E-05 8.74696815861276E-06 -0.000155511793327179"
-        rpy="0 0 0" />
-      <mass
-        value="0.774041102749819" />
-      <inertia
-        ixx="0.000555068815324583"
-        ixy="2.15732280355057E-07"
-        ixz="-1.85654347062673E-10"
-        iyy="0.000555930826369468"
-        iyz="2.27283260482476E-10"
-        izz="0.000988906210850007" />
+        xyz="-3.68604325448052E-05 8.74696815872378E-06 -0.000155511793327234"
+        rpy="0 0 0" />
+      <mass
+        value="0.77404110274982" />
+      <inertia
+        ixx="0.00055506881532458"
+        ixy="2.15732280355355E-07"
+        ixz="-1.8565434672159E-10"
+        iyy="0.000555930826369469"
+        iyz="2.2728326005673E-10"
+        izz="0.00098890621085001" />
     </inertial>
     <visual>
@@ -105,6 +105,6 @@
     type="continuous">
     <origin
-      xyz="-0.196999999999994 0.243373703143014 -0.410500520826094"
-      rpy="1.5707963267949 -0.698892577239709 1.57079632679526" />
+      xyz="0.243373703143014 0.196999999999994 -0.410500520826094"
+      rpy="1.5707963267949 -0.698892577239709 0" />
     <parent
       link="Mobile_Base" />
@@ -118,15 +118,15 @@
     <inertial>
       <origin
-        xyz="-3.83185982943957E-10 -5.66471758389753E-10 -6.83960459935129E-08"
-        rpy="0 0 0" />
-      <mass
-        value="0.0352584429300109" />
-      <inertia
-        ixx="1.04260747160857E-05"
-        ixy="-3.74985932672452E-16"
-        ixz="3.16159847322509E-11"
-        iyy="1.04260747162552E-05"
-        iyz="-7.59166287983956E-12"
-        izz="3.24617145964053E-06" />
+        xyz="-3.83179044050053E-10 -5.66471425322845E-10 -6.83960459380017E-08"
+        rpy="0 0 0" />
+      <mass
+        value="0.0352584429300114" />
+      <inertia
+        ixx="1.04260747160859E-05"
+        ixy="-3.74986144430689E-16"
+        ixz="3.16159847563384E-11"
+        iyy="1.04260747162553E-05"
+        iyz="-7.59166288672171E-12"
+        izz="3.2461714596406E-06" />
     </inertial>
     <visual>
@@ -171,15 +171,15 @@
     <inertial>
       <origin
-        xyz="-3.09857084435095E-10 1.10555134491541E-09 -4.17113807937852E-08"
-        rpy="0 0 0" />
-      <mass
-        value="0.0352584429300112" />
-      <inertia
-        ixx="1.04260761905347E-05"
-        ixy="2.10247077096114E-16"
-        ixz="-2.4788845562525E-11"
+        xyz="-3.09857084435095E-10 1.10555131715984E-09 -4.17113807937852E-08"
+        rpy="0 0 0" />
+      <mass
+        value="0.0352584429300109" />
+      <inertia
+        ixx="1.04260761905346E-05"
+        ixy="2.1024734179391E-16"
+        ixz="-2.4788845569513E-11"
         iyy="1.04260761890094E-05"
-        iyz="-2.10620761179513E-11"
-        izz="3.24617146052916E-06" />
+        iyz="-2.10620761229012E-11"
+        izz="3.2461714605291E-06" />
     </inertial>
     <visual>
@@ -224,14 +224,14 @@
     <inertial>
       <origin
-        xyz="7.28457724696874E-09 2.76751455086099E-09 2.27604661784397E-08"
-        rpy="0 0 0" />
-      <mass
-        value="0.0352584429300111" />
+        xyz="7.28457724696874E-09 2.76751460637215E-09 2.27604659563951E-08"
+        rpy="0 0 0" />
+      <mass
+        value="0.0352584429300112" />
       <inertia
         ixx="1.04260768064924E-05"
-        ixy="-1.98661171978739E-14"
-        ixz="-3.25498755598683E-11"
+        ixy="-1.98661176213904E-14"
+        ixz="-3.25498755616683E-11"
         iyy="1.04260768503918E-05"
-        iyz="-1.43134028288981E-12"
+        iyz="-1.43134028341921E-12"
         izz="3.2461715182147E-06" />
     </inertial>
@@ -277,15 +277,15 @@
     <inertial>
       <origin
-        xyz="-8.85009204809606E-10 8.87345419364749E-10 -1.82681258453776E-08"
-        rpy="0 0 0" />
-      <mass
-        value="0.035258442930011" />
-      <inertia
-        ixx="1.04260768940346E-05"
-        ixy="6.843225238284E-16"
-        ixz="-1.09712169237017E-11"
-        iyy="1.04260768941284E-05"
-        iyz="3.06406603017413E-11"
-        izz="3.24617146037589E-06" />
+        xyz="-8.85001738559765E-10 8.87343976074817E-10 -1.82681261229334E-08"
+        rpy="0 0 0" />
+      <mass
+        value="0.0352584429300108" />
+      <inertia
+        ixx="1.04260768940345E-05"
+        ixy="6.84323106163551E-16"
+        ixz="-1.09712169219895E-11"
+        iyy="1.04260768941283E-05"
+        iyz="3.06406602966855E-11"
+        izz="3.24617146037585E-06" />
     </inertial>
     <visual>
@@ -330,14 +330,14 @@
     <inertial>
       <origin
-        xyz="1.60439110885591E-08 5.69080083057116E-09 1.2380305391968E-07"
+        xyz="1.60439111440702E-08 5.69080083057116E-09 1.2380305391968E-07"
         rpy="0 0 0" />
       <mass
         value="0.035258442930011" />
       <inertia
-        ixx="1.04260694141622E-05"
-        ixy="-9.94372503073185E-14"
-        ixz="-1.26413841544385E-11"
+        ixx="1.04260694141623E-05"
+        ixy="-9.94372509425932E-14"
+        ixz="-1.26413841572443E-11"
         iyy="1.04260696259208E-05"
-        iyz="2.99325036340899E-11"
+        iyz="2.99325036380074E-11"
         izz="3.24617174875245E-06" />
     </inertial>
@@ -383,15 +383,15 @@
     <inertial>
       <origin
-        xyz="-3.825635364052E-10 -1.68518193843781E-09 4.39527294560094E-08"
-        rpy="0 0 0" />
-      <mass
-        value="0.0352584429300111" />
+        xyz="-3.82563758449805E-10 -1.68518196619338E-09 4.39527294004982E-08"
+        rpy="0 0 0" />
+      <mass
+        value="0.035258442930011" />
       <inertia
         ixx="1.04260760941714E-05"
-        ixy="-2.85658102752809E-16"
-        ixz="2.80429237954922E-11"
+        ixy="-2.85658314511046E-16"
+        ixz="2.80429237867042E-11"
         iyy="1.04260760917002E-05"
-        iyz="1.65168143921329E-11"
-        izz="3.24617146148317E-06" />
+        iyz="1.65168143896448E-11"
+        izz="3.24617146148314E-06" />
     </inertial>
     <visual>
@@ -436,5 +436,5 @@
     <inertial>
       <origin
-        xyz="4.28941293595386E-09 8.82995787598873E-10 -1.01682179981522E-07"
+        xyz="4.28941293595386E-09 8.82995843110024E-10 -1.01682180037033E-07"
         rpy="0 0 0" />
       <mass
@@ -442,9 +442,9 @@
       <inertia
         ixx="1.04260718732603E-05"
-        ixy="-4.33398087044761E-15"
-        ixz="2.94154428727412E-11"
+        ixy="-4.33397981165643E-15"
+        ixz="2.94154428780881E-11"
         iyy="1.04260718866193E-05"
-        iyz="-1.4005428896808E-11"
-        izz="3.2461714747039E-06" />
+        iyz="-1.40054288998785E-11"
+        izz="3.24617147470388E-06" />
     </inertial>
     <visual>
@@ -489,15 +489,15 @@
     <inertial>
       <origin
-        xyz="-4.45606107568608E-10 -1.68479385997955E-09 4.58650017132189E-08"
-        rpy="0 0 0" />
-      <mass
-        value="0.0352584429300115" />
-      <inertia
-        ixx="1.04260760091362E-05"
-        ixy="-3.83896454579771E-16"
-        ixz="3.22721314246384E-11"
-        iyy="1.04260760061884E-05"
-        iyz="-4.12147536543168E-12"
-        izz="3.24617146194952E-06" />
+        xyz="-4.45605996546306E-10 -1.68479385997955E-09 4.58650016577078E-08"
+        rpy="0 0 0" />
+      <mass
+        value="0.035258442930011" />
+      <inertia
+        ixx="1.0426076009136E-05"
+        ixy="-3.83896719277567E-16"
+        ixz="3.2272131431729E-11"
+        iyy="1.04260760061882E-05"
+        iyz="-4.12147536670223E-12"
+        izz="3.24617146194942E-06" />
     </inertial>
     <visual>
@@ -548,8 +548,8 @@
       <inertia
         ixx="0.000205567523367468"
-        ixy="4.86825936022437E-10"
-        ixz="5.22777710432475E-10"
+        ixy="4.86825936008885E-10"
+        ixz="5.22777710432301E-10"
         iyy="0.000205922237695722"
-        iyz="8.40224944645304E-11"
+        iyz="8.40224944649351E-11"
         izz="0.000366267561115225" />
     </inertial>
@@ -582,6 +582,6 @@
     type="continuous">
     <origin
-      xyz="-0.197 -0.243373703143012 -0.410500520826101"
-      rpy="1.5707963267949 -0.479686767241463 1.57079632679489" />
+      xyz="-0.243373703143012 0.197 -0.410500520826101"
+      rpy="1.5707963267949 -0.479686767241463 0" />
     <parent
       link="Mobile_Base" />
@@ -598,12 +598,12 @@
         rpy="0 0 0" />
       <mass
-        value="0.0352584429300112" />
+        value="0.0352584429300111" />
       <inertia
         ixx="1.04260715177521E-05"
         ixy="-2.16967544708089E-13"
-        ixz="-9.22230104291594E-12"
+        ixz="-9.22230104503352E-12"
         iyy="1.04260716218938E-05"
-        iyz="3.09410049840542E-11"
-        izz="3.24617190478417E-06" />
+        iyz="3.09410049823601E-11"
+        izz="3.24617190478418E-06" />
     </inertial>
     <visual>
@@ -648,15 +648,15 @@
     <inertial>
       <origin
-        xyz="7.42938899289669E-09 -8.73704070203374E-09 8.61521962658429E-08"
-        rpy="0 0 0" />
-      <mass
-        value="0.0352584429300108" />
-      <inertia
-        ixx="1.04260734013828E-05"
+        xyz="7.42938899289669E-09 -8.73704070203374E-09 8.61521962380873E-08"
+        rpy="0 0 0" />
+      <mass
+        value="0.0352584429300111" />
+      <inertia
+        ixx="1.04260734013829E-05"
         ixy="6.31409768982622E-14"
-        ixz="9.33284556977417E-12"
-        iyy="1.04260733892382E-05"
-        iyz="3.12763115710681E-11"
-        izz="3.2461715855996E-06" />
+        ixz="9.33284556850362E-12"
+        iyy="1.04260733892384E-05"
+        iyz="3.12763115730798E-11"
+        izz="3.24617158559965E-06" />
     </inertial>
     <visual>
@@ -860,14 +860,14 @@
     <inertial>
       <origin
-        xyz="2.33893460155343E-10 1.54178639300007E-09 -2.60845123278841E-08"
-        rpy="0 0 0" />
-      <mass
-        value="0.035258442930011" />
+        xyz="2.33893432399768E-10 1.54178633748892E-09 -2.60845123278841E-08"
+        rpy="0 0 0" />
+      <mass
+        value="0.0352584429300111" />
       <inertia
         ixx="1.04260767232418E-05"
-        ixy="-3.71422041546879E-16"
-        ixz="3.32532285718695E-12"
-        iyy="1.04260767205083E-05"
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
File: recon_bot_description/robot/robot.urdf.xacro (robot description, xacro)
@@ -25,5 +25,5 @@
         <parent link="Mobile_Base"/> <!-- Ensure Mobile_Base is defined in the included files -->
         <child link="$(arg camera_name)_camera_link"/> <!-- Ensure zed_camera_link is defined in the ZED macro -->
-        <origin xyz="0 0.265 -0.085" rpy="0 0 1.57"/>
+        <origin xyz="0.265 0 -0.085" rpy="0 0 0"/>
       </joint>
     </xacro:if>
