Commit message: jetson updated

File: recon_bot_description/robot/lidar.xacro (robot description, xacro)
@@ -4,5 +4,5 @@
         <parent link="Mobile_Base"/>
         <child link="lidar_front_link"/>
-        <origin xyz="-0.222 0.25 -0.230" rpy="0 0 0"/>
+        <origin xyz="-0.222 0.25 -0.230" rpy="3.14 0 0"/>
     </joint>
     <link name="lidar_front_link">
@@ -29,5 +29,5 @@
         <parent link="Mobile_Base"/>
         <child link="lidar_back_link"/>
-        <origin xyz="0.222 -0.25 -0.230" rpy="0 0 0"/>
+        <origin xyz="0.222 -0.25 -0.230" rpy="3.14 0 0"/>
     </joint>
     <link name="lidar_back_link">

File: recon_bot_description/robot/robot.core.xacro (robot description, xacro)
@@ -5,4 +5,12 @@
      For more information, please see http://wiki.ros.org/sw_urdf_exporter -->
   <xacro:include filename="$(find recon_bot_description)/robot/materials.xacro"/>
+  <link name="odom">
+    <origin xyz="0.0 0.0 0.0" rpy="0.0 0.0 3.14" />
+  </link>
+  <joint name="odom_to_basefootprint" type="fixed">
+    <parent link="odom"/>
+    <child link="base_footprint"/>
+    <origin rpy="0 0 0" xyz="0 0 0"/>
+  </joint>
   <link name="base_footprint">
     <origin xyz="0.0 0.0 0.0" rpy="0.0 0.0 3.14" />
@@ -51,5 +59,5 @@
     <parent link="base_footprint"/>
     <child link="Mobile_Base"/>
-    <origin rpy="0 0 0" xyz="0 0 0.4"/>
+    <origin rpy="0 0 0" xyz="0 0 0.48"/>
   </joint>
   <link

File: recon_bot_description/robot/ros2_control.xacro (robot description, xacro)
@@ -1,18 +1,6 @@
 <?xml version="1.0"?>
 <robot xmlns:xacro="http://www.ros.org/wiki/xacro">
-    <ros2_control name="RealRobot" type="system">
-        <hardware>
-            <plugin>mecanumdrive_arduino/MecanumDriveArduinoHardware</plugin>
-            <param name="left_wheel_name">J_Wheel_LF</param>
-            <param name="right_wheel_name">J_Wheel_LR</param>
-            <param name="left_wheel_name">J_Wheel_RF</param>
-            <param name="right_wheel_name">J_Wheel_RR</param>
-            <param name="loop_rate">30</param>
-            <param name="device">/dev/ttyUSB0</param>
-            <param name="baud_rate">57600</param>
-            <param name="timeout_ms">1000</param>
-            <param name="enc_counts_per_rev">3436</param>
-        </hardware>
-        <joint name="left_wheel_joint">
+    <ros2_control name="recon_bot" type="system">
+        <joint name="J_Wheel_LF">
             <command_interface name="velocity">
                 <param name="min">-10</param>
@@ -22,5 +10,5 @@
             <state_interface name="velocity"/>
         </joint>
-        <joint name="right_wheel_joint">
+        <joint name="J_Wheel_LR">
             <command_interface name="velocity">
                 <param name="min">-10</param>
@@ -30,5 +18,5 @@
             <state_interface name="velocity"/>
         </joint>
-        <joint name="right_wheel_joint">
+        <joint name="J_Wheel_RF">
             <command_interface name="velocity">
                 <param name="min">-10</param>
@@ -38,5 +26,5 @@
             <state_interface name="velocity"/>
         </joint>
-        <joint name="right_wheel_joint">
+        <joint name="J_Wheel_RR">
             <command_interface name="velocity">
                 <param name="min">-10</param>

Commit message: modify lidar origin

File: recon_bot_description/robot/lidar.xacro (robot description, xacro)
@@ -4,5 +4,5 @@
         <parent link="Mobile_Base"/>
         <child link="lidar_front_link"/>
-        <origin xyz="-0.222 0.25 -0.230" rpy="3.14 0 0"/>
+        <origin xyz="0.222 0.25 -0.230" rpy="0 0 3.14"/>
     </joint>
     <link name="lidar_front_link">
@@ -29,5 +29,5 @@
         <parent link="Mobile_Base"/>
         <child link="lidar_back_link"/>
-        <origin xyz="0.222 -0.25 -0.230" rpy="3.14 0 0"/>
+        <origin xyz="-0.222 -0.25 -0.230" rpy="0 0 3.14"/>
     </joint>
     <link name="lidar_back_link">

Commit message: update 2025

File: recon_bot_description/robot/lidar.xacro (robot description, xacro)
@@ -4,5 +4,5 @@
         <parent link="Mobile_Base"/>
         <child link="lidar_front_link"/>
-        <origin xyz="0.222 0.25 -0.230" rpy="0 0 3.14"/>
+        <origin xyz="0.222 0.25 -0.230" rpy="0 3.14 1.57"/>
     </joint>
     <link name="lidar_front_link">
@@ -29,5 +29,5 @@
         <parent link="Mobile_Base"/>
         <child link="lidar_back_link"/>
-        <origin xyz="-0.222 -0.25 -0.230" rpy="0 0 3.14"/>
+        <origin xyz="-0.222 -0.25 -0.230" rpy="0 3.13 1.57"/>
     </joint>
     <link name="lidar_back_link">

Commit message: create lidar merge

File: recon_bot_description/robot/lidar.xacro (robot description, xacro)
@@ -29,5 +29,5 @@
         <parent link="Mobile_Base"/>
         <child link="lidar_back_link"/>
-        <origin xyz="-0.222 -0.25 -0.230" rpy="0 3.13 1.57"/>
+        <origin xyz="-0.222 -0.25 -0.230" rpy="0 3.14 1.57"/>
     </joint>
     <link name="lidar_back_link">
