Commit message: ros2_control updated

File: recon_bot_description/robot/recon_bot.urdf.xacro (robot description, xacro)
@@ -2,7 +2,9 @@
 <robot xmlns:xacro="http://www.ros.org/wiki/xacro" name="recon_bot">
     <!-- Include robot and lidar Xacro files -->
-    <xacro:include filename="$(find recon_bot_description)/robot/robot.core.xacro"/>
+    <xacro:include filename="$(find recon_bot_description)/robot/recon_bot.core.xacro"/>
     <xacro:include filename="$(find recon_bot_description)/robot/lidar.xacro"/>
-    <!-- Arguments for ZED Camera -->
+    <xacro:include filename="$(find recon_bot_description)/robot/ros2_control.xacro" />
+    <xacro:recon_x_ros2_control name="recon_x_ros2_control" />
+/*<!-- Arguments for ZED Camera -->
     <xacro:arg name="camera_name" default="zed" />
     <xacro:arg name="camera_model" default="zed2i" />

File: recon_bot_description/robot/ros2_control.xacro (robot description, xacro)
@@ -1,37 +1,45 @@
 <?xml version="1.0"?>
 <robot xmlns:xacro="http://www.ros.org/wiki/xacro">
-    <ros2_control name="recon_bot" type="system">
-        <joint name="J_Wheel_LF">
-            <command_interface name="velocity">
-                <param name="min">-10</param>
-                <param name="max">10</param>
-            </command_interface>
-            <state_interface name="position"/>
-            <state_interface name="velocity"/>
-        </joint>
-        <joint name="J_Wheel_LR">
-            <command_interface name="velocity">
-                <param name="min">-10</param>
-                <param name="max">10</param>
-            </command_interface>
-            <state_interface name="position"/>
-            <state_interface name="velocity"/>
-        </joint>
-        <joint name="J_Wheel_RF">
-            <command_interface name="velocity">
-                <param name="min">-10</param>
-                <param name="max">10</param>
-            </command_interface>
-            <state_interface name="position"/>
-            <state_interface name="velocity"/>
-        </joint>
-        <joint name="J_Wheel_RR">
-            <command_interface name="velocity">
-                <param name="min">-10</param>
-                <param name="max">10</param>
-            </command_interface>
-            <state_interface name="position"/>
-            <state_interface name="velocity"/>
-        </joint>
-    </ros2_control>
+    <xacro:macro name="recon_x_ros2_control" params="name">
+        <ros2_control name="recon_bot" type="system">
+            <hardware>
+                <plugin>dynamixel_hardware/DynamixelHardware</plugin>
+                <param name="usb_port">/dev/ttyUSB_DYNAMIXEL</param>
+                <param name="baud_rate">1000000</param>
+                <!-- <param name="use_dummy">true</param> -->
+            </hardware>
+            <joint name="J_Wheel_LF">
+                <param name="id">4</param>
+                <command_interface name="position"/>
+                <command_interface name="velocity"/>
+                <state_interface name="position"/>
+                <state_interface name="velocity"/>
+                <state_interface name="effort"/>
+            </joint>
+            <joint name="J_Wheel_RF">
+                <param name="id">3</param>
+                <command_interface name="position"/>
+                <command_interface name="velocity"/>
+                <state_interface name="position"/>
+                <state_interface name="velocity"/>
+                <state_interface name="effort"/>
+            </joint>
+            <joint name="J_Wheel_LR">
+                <param name="id">2</param>
+                <command_interface name="position"/>
+                <command_interface name="velocity"/>
+                <state_interface name="position"/>
+                <state_interface name="velocity"/>
+                <state_interface name="effort"/>
+            </joint>
+            <joint name="J_Wheel_RR">
+                <param name="id">1</param>
+                <command_interface name="position"/>
+                <command_interface name="velocity"/>
+                <state_interface name="position"/>
+                <state_interface name="velocity"/>
+                <state_interface name="effort"/>
+            </joint>
+        </ros2_control>
+    </xacro:macro>
 </robot>

Commit message: code_update_dynamixel_ros2_control

File: recon_bot_description/robot/recon_bot.urdf.xacro (robot description, xacro)
@@ -9,7 +9,6 @@
     <xacro:arg name="camera_name" default="zed" />
     <xacro:arg name="camera_model" default="zed2i" />
-    <xacro:arg name="use_zed_localization" default="true" />
-    <!-- <xacro:arg name="baseline" default="0.0" /> -->
-    <xacro:arg name="custom_baseline"  default="0.0" />
+    <xacro:arg name="use_zed_localization" default="false" />
+  <xacro:arg name="custom_baseline"  default="0.0" />
     <!-- If GNSS fusion is enabled the position of the antenna with respect to the camera mount point is required -->
     <xacro:arg name="enable_gnss"   default="false" />

File: recon_bot_description/robot/ros2_control.xacro (robot description, xacro)
@@ -2,5 +2,5 @@
 <robot xmlns:xacro="http://www.ros.org/wiki/xacro">
     <xacro:macro name="recon_x_ros2_control" params="name">
-        <ros2_control name="recon_bot" type="system">
+        <ros2_control name="${name}" type="system">
             <hardware>
                 <plugin>dynamixel_hardware/DynamixelHardware</plugin>
@@ -9,35 +9,27 @@
                 <!-- <param name="use_dummy">true</param> -->
             </hardware>
-            <joint name="J_Wheel_LF">
-                <param name="id">4</param>
-                <command_interface name="position"/>
+            <joint name="J_Wheel_RR">
+                <param name="id">1</param>
                 <command_interface name="velocity"/>
                 <state_interface name="position"/>
                 <state_interface name="velocity"/>
-                <state_interface name="effort"/>
+            </joint>
+            <joint name="J_Wheel_LR">
+                <param name="id">2</param>
+                <command_interface name="velocity"/>
+                <state_interface name="position"/>
+                <state_interface name="velocity"/>
             </joint>
             <joint name="J_Wheel_RF">
                 <param name="id">3</param>
-                <command_interface name="position"/>
                 <command_interface name="velocity"/>
                 <state_interface name="position"/>
                 <state_interface name="velocity"/>
-                <state_interface name="effort"/>
             </joint>
-            <joint name="J_Wheel_LR">
-                <param name="id">2</param>
-                <command_interface name="position"/>
+            <joint name="J_Wheel_LF">
+                <param name="id">4</param>
                 <command_interface name="velocity"/>
                 <state_interface name="position"/>
                 <state_interface name="velocity"/>
-                <state_interface name="effort"/>
-            </joint>
-            <joint name="J_Wheel_RR">
-                <param name="id">1</param>
-                <command_interface name="position"/>
-                <command_interface name="velocity"/>
-                <state_interface name="position"/>
-                <state_interface name="velocity"/>
-                <state_interface name="effort"/>
             </joint>
         </ros2_control>

Commit message: launch file name updated

File: recon_bot_description/robot/recon_bot.urdf.xacro (robot description, xacro)
@@ -9,5 +9,5 @@
     <!-- Arguments for ZED Camera -->
     <xacro:arg name="camera_name" default="zed" />
-    <xacro:arg name="camera_model" default="zed2i" />
+    <xacro:arg name="camera_model" default="zed2" />
     <xacro:arg name="use_zed_localization" default="false" />
     <xacro:arg name="custom_baseline"  default="0.0" />
@@ -35,5 +35,5 @@
         <parent link="Mobile_Base"/>
         <child link="$(arg camera_name)_camera_link"/>
-        <origin xyz="0 0.265 -0.085" rpy="0 0 1.57"/>
+        <origin xyz="0.265 0 -0.085" rpy="0 0 0"/>
       </joint>
     </xacro:unless>
