Commit message: slam and nav updated

File: recon_bot_description/robot/Recon_Mobile_Base_.urdf (robot description, URDF)
Before this commit: robot recon_bot_description, 41 links, 40 joints
Joints:
- removed joint odom_to_basefootprint
- added joint odom_to_base_footprint: type fixed, parent odom, child base_footprint, origin xyz=0 0 0 rpy=0 0 0

File: recon_bot_description/robot/robot.urdf.xacro (robot description, xacro)
@@ -4,5 +4,5 @@
     <xacro:include filename="$(find recon_bot_description)/robot/robot.core.xacro"/>
     <xacro:include filename="$(find recon_bot_description)/robot/lidar.xacro"/>
-    Arguments for ZED Camera
+    <!-- Arguments for ZED Camera -->
     <xacro:arg name="camera_name" default="zed" />
     <xacro:arg name="camera_model" default="zed2i" />

Commit message: VIO_EKF updated

File: recon_bot_description/robot/Recon_Mobile_Base_.urdf (robot description, URDF)
Before this commit: robot recon_bot_description, 41 links, 40 joints
Links:
- removed link base_footprint
- removed link odom
Joints:
- removed joint basefootprint_to_base
- removed joint odom_to_base_footprint

File: recon_bot_description/robot/Recon_Mobile_Base_visual.urdf (robot description, URDF)
Before this commit: robot recon_bot_description, 41 links, 40 joints
Joints:
- removed joint basefootprint_to_base

File: recon_bot_description/robot/recon_bot.core.xacro (robot description, xacro)
@@ -16,5 +16,5 @@
     <origin xyz="0.0 0.0 0.0" rpy="0.0 0.0 3.14" />
   </link>
-    <joint name="base_footprint_to_Mobile_Base" type="fixed">
+    <joint name="Mobile_Base_to_base_footprint" type="fixed">
     <parent link="base_footprint"/>
     <child link="Mobile_Base"/>
@@ -22,5 +22,5 @@
   </joint>
   <link
-    name="Mobile_Base">
+    name="Mobile_Base"> <!-- name_of_my_robot_base_link -->
     <inertial>
       <origin
@@ -65,5 +65,5 @@
     <parent link="Mobile_Base"/>
     <child link="merged_scan_frame"/>
-    <origin xyz="0 0 -0.2" rpy="0 0 0"/>
+    <origin xyz="0 0 -0.3" rpy="0 0 0"/>
   </joint>
   <link

File: recon_bot_description/robot/recon_bot.urdf.xacro (robot description, xacro)
@@ -7,8 +7,7 @@
     <xacro:recon_control name="recon_control" />
     <!-- Arguments for ZED Camera -->
-    <!-- Arguments for ZED Camera -->
     <xacro:arg name="camera_name" default="zed" />
     <xacro:arg name="camera_model" default="zed2" />
-    <xacro:arg name="use_zed_localization" default="false" />
+    <xacro:arg name="use_zed_localization" default="false" /> <!-- สำคัญ! -->
     <xacro:arg name="custom_baseline"  default="0.0" />
     <!-- If GNSS fusion is enabled the position of the antenna with respect to the camera mount point is required -->
@@ -23,13 +22,13 @@
     <!-- Joint to connect the ZED Camera to the robot -->
     <xacro:if value="$(arg use_zed_localization)">
-      <!-- ZED Localization: camera_link is the parent, Mobile_Base is the child -->
+      <!-- ZED Localization: camera_link is the parent, Mobile_Base is the child --> <!-- กรณีใช้ ZED เป็น localization หลัก (ไม่แนะนำ) -->
       <joint name="$(arg camera_name)_joint" type="fixed">
-        <parent link="Mobile_Base"/> <!-- Ensure Mobile_Base is defined in the included files -->
-        <child link="$(arg camera_name)_camera_link"/> <!-- Ensure zed_camera_link is defined in the ZED macro -->
-        <origin xyz="0.265 0 -0.085" rpy="0 0 0"/>
+        <parent link="$(arg camera_name)_camera_link"/> <!-- Ensure Mobile_Base is defined in the included files -->
+        <child link="Mobile_Base"/> <!-- Ensure zed_camera_link is defined in the ZED macro -->
+        <origin xyz="-0.265 0 0.085" rpy="0 0 0"/>
       </joint>
     </xacro:if>
     <xacro:unless value="$(arg use_zed_localization)">
-      <!-- No ZED Localization: camera_link is the child, Mobile_Base is the parent -->
+      <!-- No ZED Localization: camera_link is the child, Mobile_Base is the parent --> <!-- กรณีใช้ VIO + EKF (แนะนำ) -->
       <joint name="$(arg camera_name)_joint" type="fixed">
         <parent link="Mobile_Base"/>

File: recon_bot_description/robot/zed_macro.urdf.xacro (robot description, xacro)
@@ -129,39 +129,4 @@
       <origin xyz="${optical_offset_x} ${baseline/2} 0" rpy="0 0 0" />
     </joint>
-    <link name="${name}_left_camera_optical_frame"/>
-    <joint name="${name}_left_camera_optical_joint" type="fixed">
-      <origin xyz="0 0 0" rpy="-${M_PI/2} 0.0 -${M_PI/2}"/>
-      <parent link="${name}_left_camera_frame"/>
-      <child link="${name}_left_camera_optical_frame"/>
-    </joint>
-    <!-- Right Camera -->
-    <link name="${name}_right_camera_frame">
-      <xacro:if value="${model == 'virtual'}">
-        <visual>
-          <origin xyz="0 0 0" rpy="0 0 0"/>
-          <geometry>
-            <mesh filename="package://zed_interfaces/meshes/${model}.stl" />
-          </geometry>
-          <material name="${model}_mat" />
-        </visual>
-        <collision>
-          <origin xyz="0 0 0" rpy="0 0 0"/>
-          <geometry>
-            <mesh filename="package://zed_interfaces/meshes/${model}.stl" />
-          </geometry>
-        </collision>
-      </xacro:if>
-    </link>
-    <joint name="${name}_right_camera_joint" type="fixed">
-      <parent link="${name}_camera_center"/>
-      <child link="${name}_right_camera_frame"/>
-      <origin xyz="${optical_offset_x} -${baseline/2} 0" rpy="0 0 0" />
-    </joint>
-    <link name="${name}_right_camera_optical_frame"/>
-    <joint name="${name}_right_camera_optical_joint" type="fixed">
-      <origin xyz="0 0 0" rpy="-${M_PI/2} 0.0 -${M_PI/2}"/>
-      <parent link="${name}_right_camera_frame"/>
-      <child link="${name}_right_camera_optical_frame"/>
-    </joint>
     <!-- ZED2 Sensors -->
     <xacro:if value="${model == 'zed2'}">
