Commit message: update 17052025

File: recon_bot_description/robot/recon_bot.core.xacro (robot description, xacro)
@@ -5,5 +5,5 @@
      For more information, please see http://wiki.ros.org/sw_urdf_exporter -->
   <xacro:include filename="$(find recon_bot_description)/robot/materials.xacro"/>
-  <link name="odom">
+  <!-- <link name="odom">
     <origin xyz="0.0 0.0 0.0" rpy="0.0 0.0 3.14" />
   </link>
@@ -12,5 +12,5 @@
     <child link="base_footprint"/>
     <origin rpy="0 0 0" xyz="0 0 0"/>
-  </joint>
+  </joint> -->
   <link name="base_footprint">
     <origin xyz="0.0 0.0 0.0" rpy="0.0 0.0 3.14" />
@@ -46,7 +46,5 @@
       </geometry>
       <material
-        name="">
-        <color
-          rgba="0.792156862745098 0.819607843137255 0.933333333333333 1" />
+        name="orange">
       </material>
     </visual>
@@ -156,5 +154,5 @@
   <joint
     name="J_Roller_LF_1"
-    type="continuous">
+    type="fixed">
     <origin
       xyz="0.0495000000000021 0 0"
@@ -209,5 +207,5 @@
   <joint
     name="J_Roller_LF_2"
-    type="continuous">
+    type="fixed">
     <origin
       xyz="0.0350017856687387 0.0350017856687551 0"
@@ -262,5 +260,5 @@
   <joint
     name="J_Roller_LF_3"
-    type="continuous">
+    type="fixed">
     <origin
       xyz="0 0.0494999999999665 0"
@@ -315,5 +313,5 @@
   <joint
     name="J_Roller_LF_4"
-    type="continuous">
+    type="fixed">
     <origin
       xyz="-0.0350017856687272 0.0350017856687195 0"
@@ -368,5 +366,5 @@
   <joint
     name="J_Roller_LF_5"
-    type="continuous">
+    type="fixed">
     <origin
       xyz="-0.0495000000000251 0 0"
@@ -421,5 +419,5 @@
   <joint
     name="J_Roller_LF_6"
-    type="continuous">
+    type="fixed">
     <origin
       xyz="-0.0350017856687449 -0.0350017856687672 0"
@@ -474,5 +472,5 @@
   <joint
     name="J_Roller_LF_7"
-    type="continuous">
+    type="fixed">
     <origin
       xyz="0 -0.0494999999999995 0"
@@ -527,5 +525,5 @@
   <joint
     name="J_Roller_LF_8"
-    type="continuous">
+    type="fixed">
     <origin
       xyz="0.0350017856687419 -0.0350017856687232 0"
@@ -633,5 +631,5 @@
   <joint
     name="J_Roller_LR_1"
-    type="continuous">
+    type="fixed">
     <origin
       xyz="0.0494999999999991 0 0"
@@ -686,5 +684,5 @@
   <joint
     name="J_Roller_LR_2"
-    type="continuous">
+    type="fixed">
     <origin
       xyz="0.0350017856687349 0.0350017856687338 0"
@@ -739,5 +737,5 @@
   <joint
     name="J_Roller_LR_3"
-    type="continuous">
+    type="fixed">
     <origin
       xyz="0 0.0494999999999999 0"
@@ -792,5 +790,5 @@
   <joint
     name="J_Roller_LR_4"
-    type="continuous">
+    type="fixed">
     <origin
       xyz="-0.0350017856687312 0.035001785668738 0"
@@ -845,5 +843,5 @@
   <joint
     name="J_Roller_LR_5"
-    type="continuous">
+    type="fixed">
     <origin
       xyz="-0.0494999999999998 0 0"
@@ -898,5 +896,5 @@
   <joint
     name="J_Roller_LR_6"
-    type="continuous">
+    type="fixed">
     <origin
       xyz="-0.0350017856687373 -0.035001785668729 0"
@@ -951,5 +949,5 @@
   <joint
     name="J_Roller_LR_7"
-    type="continuous">
+    type="fixed">
     <origin
       xyz="0 -0.0494999999999981 0"
@@ -1004,5 +1002,5 @@
   <joint
     name="J_Roller_LR_8"
-    type="continuous">
+    type="fixed">
     <origin
       xyz="0.0350017856687324 -0.035001785668733 0"
@@ -1110,5 +1108,5 @@
   <joint
     name="J_Roller_RF_1"
-    type="continuous">
+    type="fixed">
     <origin
       xyz="0.0494999999999999 0 0"
@@ -1163,5 +1161,5 @@
   <joint
     name="J_Roller_RF_2"
-    type="continuous">
+    type="fixed">
     <origin
       xyz="0.0350017856687338 -0.0350017856687341 0"
@@ -1216,5 +1214,5 @@
   <joint
     name="J_Roller_RF_3"
-    type="continuous">
+    type="fixed">
     <origin
       xyz="0 -0.0495 0"
@@ -1269,5 +1267,5 @@
   <joint
     name="J_Roller_RF_4"
-    type="continuous">
+    type="fixed">
     <origin
       xyz="-0.0350017856687344 -0.0350017856687337 0"
@@ -1322,5 +1320,5 @@
   <joint
     name="J_Roller_RF_5"
-    type="continuous">
+    type="fixed">
     <origin
       xyz="-0.0495 0 0"
@@ -1375,5 +1373,5 @@
   <joint
     name="J_Roller_RF_6"
-    type="continuous">
+    type="fixed">
     <origin
       xyz="-0.0350017856687347 0.035001785668734 0"
@@ -1428,5 +1426,5 @@
   <joint
     name="J_Roller_RF_7"
-    type="continuous">
+    type="fixed">
     <origin
       xyz="0 0.0495 0"
@@ -1481,5 +1479,5 @@
   <joint
     name="J_Roller_RF_8"
-    type="continuous">
+    type="fixed">
     <origin
       xyz="0.0350017856687329 0.0350017856687334 0"
@@ -1587,5 +1585,5 @@
   <joint
     name="J_Roller_RR_1"
-    type="continuous">
+    type="fixed">
     <origin
       xyz="0.049500000000006 0 0"
@@ -1640,5 +1638,5 @@
   <joint
     name="J_Roller_RR_2"
-    type="continuous">
+    type="fixed">
     <origin
       xyz="0.049500000000006 0 0"
@@ -1693,5 +1691,5 @@
   <joint
     name="J_Roller_RR_3"
-    type="continuous">
+    type="fixed">
     <origin
       xyz="0 -0.0495000000000001 0"
@@ -1746,5 +1744,5 @@
   <joint
     name="J_Roller_RR_4"
-    type="continuous">
+    type="fixed">
     <origin
       xyz="-0.0350017856687443 -0.0350017856687639 0"
@@ -1799,5 +1797,5 @@
   <joint
     name="J_Roller_RR_5"
-    type="continuous">
+    type="fixed">
     <origin
       xyz="-0.0495000000000206 0 0"
@@ -1852,5 +1850,5 @@
   <joint
     name="J_Roller_RR_6"
-    type="continuous">
+    type="fixed">
     <origin
       xyz="-0.0350017856687212 0.0350017856687237 0"
@@ -1905,5 +1903,5 @@
   <joint
     name="J_Roller_RR_7"
-    type="continuous">
+    type="fixed">
     <origin
       xyz="0 0.0494999999999669 0"
@@ -1958,5 +1956,5 @@
   <joint
     name="J_Roller_RR_8"
-    type="continuous">
+    type="fixed">
     <origin
       xyz="0.0350017856687396 0.0350017856687503 0"
@@ -2011,5 +2009,5 @@
   <joint
     name="J_Pin_Head_L"
-    type="prismatic">
+    type="fixed">
     <origin
       xyz="0.04 0.2352 0.06"
@@ -2069,5 +2067,5 @@
   <joint
     name="J_Pin_Head_R"
-    type="prismatic">
+    type="fixed">
     <origin
       xyz="-0.04 -0.2335 0.06"

File: recon_bot_description/robot/recon_bot.urdf.xacro (robot description, xacro)
@@ -5,5 +5,5 @@
     <xacro:include filename="$(find recon_bot_description)/robot/lidar.xacro"/>
     <xacro:include filename="$(find recon_bot_description)/robot/ros2_control.xacro" />
-    <xacro:recon_x_ros2_control name="recon_x_ros2_control" />
+    <xacro:recon_control name="recon_control" />
 /*<!-- Arguments for ZED Camera -->
     <xacro:arg name="camera_name" default="zed" />

File: recon_bot_description/robot/ros2_control.xacro (robot description, xacro)
@@ -1,10 +1,10 @@
 <?xml version="1.0"?>
 <robot xmlns:xacro="http://www.ros.org/wiki/xacro">
-    <xacro:macro name="recon_x_ros2_control" params="name">
+    <xacro:macro name="recon_control" params="name">
         <ros2_control name="${name}" type="system">
             <hardware>
                 <plugin>dynamixel_hardware/DynamixelHardware</plugin>
                 <param name="usb_port">/dev/ttyUSB_DYNAMIXEL</param>
-                <param name="baud_rate">1000000</param>
+                <param name="baud_rate">57600</param>
                 <!-- <param name="use_dummy">true</param> -->
             </hardware>

Commit message: joy and lidar caribation updated

File: recon_bot_description/robot/recon_bot.core.xacro (robot description, xacro)
@@ -59,4 +59,12 @@
     </collision>
   </link>
+    <!-- Joint and Link for the Merged Laser Scan Frame -->
+  <link name="merged_scan_frame">
+  </link>
+  <joint name="merged_scan_joint" type="fixed">
+    <parent link="Mobile_Base"/>
+    <child link="merged_scan_frame"/>
+    <origin xyz="0 0 -0.2" rpy="0 0 0"/>
+  </joint>
   <link
     name="Wheel_LF">

Commit message: meshes updated

File: recon_bot_description/robot/recon_bot.core.xacro (robot description, xacro)
@@ -43,5 +43,5 @@
       <geometry>
         <mesh
-          filename="package://recon_bot_description/meshes/Mobile_Base.STL" />
+          filename="package://recon_bot_description/meshes2/Mobile_Base_visual.stl" />
       </geometry>
       <material
@@ -89,5 +89,5 @@
       <geometry>
         <mesh
-          filename="package://recon_bot_description/meshes/Wheel_LF.STL" />
+          filename="package://recon_bot_description/meshes2/Wheel_LF_visual.stl" />
       </geometry>
       <material
@@ -566,5 +566,5 @@
       <geometry>
         <mesh
-          filename="package://recon_bot_description/meshes/Wheel_LR.STL" />
+          filename="package://recon_bot_description/meshes2/Wheel_LR_visual.stl" />
       </geometry>
       <material
@@ -1043,5 +1043,5 @@
       <geometry>
         <mesh
-          filename="package://recon_bot_description/meshes/Wheel_RF.STL" />
+          filename="package://recon_bot_description/meshes2/Wheel_RF_visual.stl" />
       </geometry>
       <material
@@ -1520,5 +1520,5 @@
       <geometry>
         <mesh
-          filename="package://recon_bot_description/meshes/Wheel_RR.STL" />
+          filename="package://recon_bot_description/meshes2/Wheel_RR_visual.stl" />
       </geometry>
       <material
@@ -1997,5 +1997,5 @@
       <geometry>
         <mesh
-          filename="package://recon_bot_description/meshes/Pin_Head_L.STL" />
+          filename="package://recon_bot_description/meshes2/Pin_Head_L_visual.stl" />
       </geometry>
       <material
@@ -2055,5 +2055,5 @@
       <geometry>
         <mesh
-          filename="package://recon_bot_description/meshes/Pin_Head_R.STL" />
+          filename="package://recon_bot_description/meshes2/Pin_Head_R_visual.stl" />
       </geometry>
       <material

File: recon_bot_description/robot/recon_bot.urdf2.xacro (robot description, xacro)
@@ -2,19 +2,13 @@
 <robot xmlns:xacro="http://www.ros.org/wiki/xacro" name="recon_bot">
     <!-- Include robot and lidar Xacro files -->
-    <xacro:include filename="$(find recon_bot_description)/robot/recon_bot.core.xacro"/>
+    <xacro:include filename="$(find recon_bot_description)/robot/recon_bot.core2.xacro"/>
     <xacro:include filename="$(find recon_bot_description)/robot/lidar.xacro"/>
     <xacro:include filename="$(find recon_bot_description)/robot/ros2_control.xacro" />
     <xacro:recon_control name="recon_control" />
-<<<<<<< Updated upstream
+    <!-- Arguments for ZED Camera -->
     <!-- Arguments for ZED Camera -->
     <xacro:arg name="camera_name" default="zed" />
     <xacro:arg name="camera_model" default="zed2" />
-    <xacro:arg name="use_zed_localization" default="false" /> <!-- สำคัญ! -->
-=======
-    <!-- Arguments for ZED Camera -->
-    <xacro:arg name="camera_name" default="zed" />
-    <xacro:arg name="camera_model" default="zed2i" />
     <xacro:arg name="use_zed_localization" default="false" />
->>>>>>> Stashed changes
     <xacro:arg name="custom_baseline"  default="0.0" />
     <!-- If GNSS fusion is enabled the position of the antenna with respect to the camera mount point is required -->
@@ -29,13 +23,13 @@
     <!-- Joint to connect the ZED Camera to the robot -->
     <xacro:if value="$(arg use_zed_localization)">
-      <!-- ZED Localization: camera_link is the parent, Mobile_Base is the child --> <!-- กรณีใช้ ZED เป็น localization หลัก (ไม่แนะนำ) -->
+      <!-- ZED Localization: camera_link is the parent, Mobile_Base is the child -->
       <joint name="$(arg camera_name)_joint" type="fixed">
-        <parent link="$(arg camera_name)_camera_link"/> <!-- Ensure Mobile_Base is defined in the included files -->
-        <child link="Mobile_Base"/> <!-- Ensure zed_camera_link is defined in the ZED macro -->
-        <origin xyz="-0.265 0 0.085" rpy="0 0 0"/>
+        <parent link="Mobile_Base"/> <!-- Ensure Mobile_Base is defined in the included files -->
+        <child link="$(arg camera_name)_camera_link"/> <!-- Ensure zed_camera_link is defined in the ZED macro -->
+        <origin xyz="0.265 0 -0.085" rpy="0 0 0"/>
       </joint>
     </xacro:if>
     <xacro:unless value="$(arg use_zed_localization)">
-      <!-- No ZED Localization: camera_link is the child, Mobile_Base is the parent --> <!-- กรณีใช้ VIO + EKF (แนะนำ) -->
+      <!-- No ZED Localization: camera_link is the child, Mobile_Base is the parent -->
       <joint name="$(arg camera_name)_joint" type="fixed">
         <parent link="Mobile_Base"/>
