Commit message: update for jetson2

File: recon_bot_description/robot/recon_bot.core2.xacro (robot description, xacro)
@@ -395,3 +395,10 @@
       velocity="0" />
   </joint>
+  <!-- World frame (root for TF tree) -->
+<link name="world"/>
+<joint name="world_to_map" type="fixed">
+  <parent link="world"/>
+  <child link="map"/>
+  <origin xyz="0 0 0" rpy="0 0 0"/>
+</joint>
 </robot>

Commit message: open_loop testing updated

File: recon_bot_description/robot/recon_bot.core2.xacro (robot description, xacro)
@@ -396,9 +396,9 @@
   </joint>
   <!-- World frame (root for TF tree) -->
-<link name="world"/>
+<!-- <link name="world"/>
 <joint name="world_to_map" type="fixed">
   <parent link="world"/>
   <child link="map"/>
   <origin xyz="0 0 0" rpy="0 0 0"/>
-</joint>
+</joint> -->
 </robot>
